Commit message: changed the link "intermediary" to "root" in order ot keep names consistent

File: combined/urdf/combined.urdf.xacro (robot description, xacro)
@@ -9,5 +9,5 @@
   <husky />
   <!-- initialize kinova with connection to top of husky-->
-  <link name="intermediary">
+  <link name="root">
     <visual>
       <origin xyz="0 0 0" rpy="0 0 0" />
@@ -25,10 +25,10 @@
   </link>
   <!-- 13.2 inches to the top center of the side plate -->
-  <joint name="intermediary_between_husky_and_kinova" type="fixed">
-    <child link="intermediary" />
+  <joint name="root_between_husky_and_kinova" type="fixed">
+    <child link="root" />
     <parent link="top_plate_link" />
     <origin xyz="0.2 0 0" rpy="0 0 3.14" />
   </joint>
-  <xacro:property name="robot_root" value="intermediary" />
+  <xacro:property name="robot_root" value="root" />
   <xacro:j2n6s300 base_parent="${robot_root}" prefix="j2n6s300" />
 </robot>

Commit message: Working on launch files for combined drive base and manipulator

File: combined/urdf/combined.urdf.xacro (robot description, xacro)
@@ -28,5 +28,5 @@
     <child link="root" />
     <parent link="top_plate_link" />
-    <origin xyz="0.2 0 0" rpy="0 0 3.14" />
+    <origin xyz="0.2 0 0" rpy="0 0 1.57" />
   </joint>
   <xacro:property name="robot_root" value="root" />

Commit message: Corresponding fixes with the depth camera in kinova description

File: combined/urdf/combined.urdf.xacro (robot description, xacro)
@@ -11,5 +11,5 @@
   <link name="root">
     <visual>
-      <origin xyz="0 0 0" rpy="0 0 0" />
+      <origin xyz="0 0 0" rpy="0 0 1.57" />
       <geometry>
         <box size = "0.00001 0.00001 0.00001"/>
